Commit message: Initial Jazzy Port (#58)
* Updated dependencies for Jazzy version

Signed-off-by: Abhishekh Reddy <helloarm@pm.me>

* Updated to new robot config

Signed-off-by: Abhishekh Reddy <helloarm@pm.me>

* Updated parameters

Signed-off-by: Abhishekh Reddy <helloarm@pm.me>

* Updated to use stamped velocities, changes to remappings, added proton...

Signed-off-by: Abhishekh Reddy <helloarm@pm.me>

* Updated dependencies

Signed-off-by: Abhishekh Reddy <helloarm@pm.me>

* Updated URDF

Signed-off-by: Abhishekh Reddy <helloarm@pm.me>

* Disabled ground segmentation just for now

Signed-off-by: Abhishekh Reddy <helloarm@pm.me>

* Removed local copies

Signed-off-by: Abhishekh Reddy <helloarm@pm.me>

* Fixed remappings

Signed-off-by: Abhishekh Reddy <helloarm@pm.me>

* Now passing correct control parameter

Signed-off-by: Abhishekh Reddy <helloarm@pm.me>

* Restored some old comments, links and mounts fields

Signed-off-by: Abhishekh Reddy <helloarm@pm.me>

* Reverted non-functional changes

Signed-off-by: Abhishekh Reddy <helloarm@pm.me>

* Removed some commented stuff and reverted a small change

Signed-off-by: Abhishekh Reddy <helloarm@pm.me>

* Re-enabled patchworkpp, works now

Signed-off-by: Abhishekh Reddy <helloarm@pm.me>

* Resolved merge conflict

Signed-off-by: Abhishekh Reddy <helloarm@pm.me>

* Resolved merge conflict and reverted includes order

Signed-off-by: Abhishekh Reddy <helloarm@pm.me>

* Fixed linting issues

Signed-off-by: Abhishekh Reddy <helloarm@pm.me>

* Fixed linting issue

Signed-off-by: Abhishekh Reddy <helloarm@pm.me>

* Removed redundant remappings for controller

Signed-off-by: Abhishekh Reddy <helloarm@pm.me>

* Fixed linting issue

Signed-off-by: Abhishekh Reddy <helloarm@pm.me>

---------

Signed-off-by: Abhishekh Reddy <helloarm@pm.me>

File: honeybee_description/urdf/honeybee_description.urdf.xacro (robot description, xacro)
@@ -17,5 +17,5 @@
   <xacro:include filename="$(find clearpath_platform_description)/urdf/j100/attachments/top_plate.urdf.xacro"/>
   <!-- Clearpath base platform -->
-  <xacro:j100 wheel="default"/>
+  <xacro:j100 control="diff_4wd" front_wheels="outdoor" rear_wheels="outdoor"/>
   <xacro:fender name="front_fender" model="default" parent_link="base_link">
     <origin xyz="0.0 0.0 0.0" rpy="0.0 0.0 0.0"/>

File: honeybee_description/urdf/includes/j100.urdf.xacro (robot description, xacro)
@@ -2,9 +2,9 @@
 <robot name="j100"
   xmlns:xacro="http://www.ros.org/wiki/xacro">
-  <xacro:include filename="$(find clearpath_platform_description)/urdf/j100/wheels/wheel.urdf.xacro"/>
   <xacro:arg name="is_sim" default="false" />
   <xacro:arg name="prefix" default="" />
   <xacro:arg name="namespace" default="" />
   <xacro:arg name="gazebo_controllers" default="$(find clearpath_control)/config/j100/control.yaml"/>
+  <xacro:arg name="use_platform_controllers" default="true"/>
   <xacro:property name="PI" value="3.1415926535897931" />
   <xacro:property name="wheelbase" value="0.262" />
@@ -12,6 +12,4 @@
   <xacro:property name="wheel_vertical_offset" value="0.0345" />
   <xacro:property name="footprint_vertical_offset" value="-0.0655" />
-  <xacro:property name="wheel_radius" value="0.098" />
-  <xacro:property name="wheel_width" value="0.040" />
   <xacro:property name="chassis_length" value="0.420" />
   <xacro:property name="chassis_width" value="0.310" />
@@ -19,45 +17,5 @@
   <xacro:property name="dummy_inertia" value="1e-09"/>
   <xacro:property name="mount_spacing" value="0.120" />
-  <xacro:macro name="j100" params="wheel:='default'">
-    <xacro:j100_wheel prefix="front_left">
-      <origin xyz="${wheelbase/2} ${track/2} ${wheel_vertical_offset}" rpy="0 0 0" />
-    </xacro:j100_wheel>
-    <xacro:j100_wheel prefix="front_right">
-      <origin xyz="${wheelbase/2} ${-track/2} ${wheel_vertical_offset}" rpy="0 0 0" />
-    </xacro:j100_wheel>
-    <xacro:j100_wheel prefix="rear_left">
-      <origin xyz="${-wheelbase/2} ${track/2} ${wheel_vertical_offset}" rpy="0 0 0" />
-    </xacro:j100_wheel>
-    <xacro:j100_wheel prefix="rear_right">
-      <origin xyz="${-wheelbase/2} ${-track/2} ${wheel_vertical_offset}" rpy="0 0 0" />
-    </xacro:j100_wheel>
-    <gazebo>
-      <plugin filename="libignition-gazebo-wheel-slip-system.so" name="ignition::gazebo::systems::WheelSlip">
-        <wheel link_name="front_left_wheel_link">
-          <slip_compliance_lateral>1.0</slip_compliance_lateral>
-          <slip_compliance_longitudinal>1.0</slip_compliance_longitudinal>
-          <wheel_normal_force>40</wheel_normal_force>
-          <wheel_radius>${wheel_radius}</wheel_radius>
-        </wheel>
-        <wheel link_name="front_right_wheel_link">
-          <slip_compliance_lateral>1.0</slip_compliance_lateral>
-          <slip_compliance_longitudinal>1.0</slip_compliance_longitudinal>
-          <wheel_normal_force>40</wheel_normal_force>
-          <wheel_radius>${wheel_radius}</wheel_radius>
-        </wheel>
-        <wheel link_name="rear_left_wheel_link">
-          <slip_compliance_lateral>1.0</slip_compliance_lateral>
-          <slip_compliance_longitudinal>1.0</slip_compliance_longitudinal>
-          <wheel_normal_force>40</wheel_normal_force>
-          <wheel_radius>${wheel_radius}</wheel_radius>
-        </wheel>
-        <wheel link_name="rear_right_wheel_link">
-          <slip_compliance_lateral>1.0</slip_compliance_lateral>
-          <slip_compliance_longitudinal>1.0</slip_compliance_longitudinal>
-          <wheel_normal_force>40</wheel_normal_force>
-          <wheel_radius>${wheel_radius}</wheel_radius>
-        </wheel>
-      </plugin>
-    </gazebo>
+  <xacro:macro name="j100" params="control:='diff_4wd' front_wheels:='outdoor' rear_wheels:='outdoor'">
     <link name="base_link"></link>
     <joint name="base_link_joint" type="fixed">
@@ -86,4 +44,25 @@
       </inertial>
     </link>
+    <!-- Add wheels -->
+    <xacro:include filename="$(find clearpath_platform_description)/urdf/j100/drivetrain/wheels.urdf.xacro"/>
+    <xacro:j100_drivetrain_wheels front_wheels="${front_wheels}" rear_wheels="${rear_wheels}"/>
+    <!-- Add drivetrain -->
+    <xacro:include filename="$(find clearpath_platform_description)/urdf/generic/drivetrain/drivetrain.urdf.xacro"/>
+    <!-- Hardware  -->
+    <xacro:if value="$(arg is_sim)">
+      <xacro:property name="hardware_plugin" value="gz_ros2_control/GazeboSimSystem"/>
+    </xacro:if>
+    <xacro:unless value="$(arg is_sim)">
+      <xacro:property name="hardware_plugin" value="clearpath_hardware_interfaces/J100Hardware"/>
+    </xacro:unless>
+    <xacro:if value="$(arg use_platform_controllers)">
+      <xacro:generic_drivetrain
+        name="j100"
+        control="${control}"
+        front_wheels="${front_wheels}"
+        rear_wheels="${rear_wheels}"
+        hardware_plugin="${hardware_plugin}"
+      />
+    </xacro:if>
     <link name="imu_0_link">
       <inertial>
@@ -102,5 +81,5 @@
         <update_rate>50</update_rate>
         <visualize>true</visualize>
-        <ignition_frame_id>imu_0_link</ignition_frame_id>
+        <gz_frame_id>imu_0_link</gz_frame_id>
         <topic>sensors/imu_0/data_raw</topic> <!-- Steve mod: have topic point somewhere reasonable -->
       </sensor>
@@ -124,5 +103,5 @@
         <always_on>1</always_on>
         <update_rate>10</update_rate>
-        <ignition_frame_id>gps_0_link</ignition_frame_id>
+        <gz_frame_id>gps_0_link</gz_frame_id>
         <topic>sensors/gps_0/fix</topic>
       </sensor>
@@ -146,62 +125,4 @@
       <origin xyz="${mount_spacing} 0 0" />
     </joint>
-    <!-- Gazebo Controller -->
-    <!-- <xacro:include filename="$(find clearpath_platform_description)/urdf/generic/gazebo.urdf.xacro"/> -->
-    <xacro:if value="$(arg is_sim)">
-      <gazebo>
-        <plugin filename="libign_ros2_control-system.so" name="ign_ros2_control::IgnitionROS2ControlPlugin">
-          <parameters>$(arg gazebo_controllers)</parameters>
-          <ros>
-            <remapping>~/odom:=platform/odom</remapping>
-            <remapping>~/cmd_vel_unstamped:=platform/cmd_vel_unstamped</remapping>
-            <remapping>/tf:=tf</remapping>
-            <remapping>/tf_static:=tf_static</remapping>
-            <remapping>/dynamic_joint_states:=platform/dynamic_joint_states</remapping>
-            <remapping>/diagnostics:=diagnostics</remapping>
-            <remapping>joint_states:=platform/joint_states</remapping>
-            <namespace>$(arg namespace)</namespace>
-          </ros>
-        </plugin>
-      </gazebo>
-      <gazebo>
-        <plugin filename="libignition-gazebo-pose-publisher-system.so" name="ignition::gazebo::systems::PosePublisher">
-          <publish_link_pose>true</publish_link_pose>
-          <publish_nested_model_pose>true</publish_nested_model_pose>
-          <use_pose_vector_msg>true</use_pose_vector_msg>
-          <update_frequency>50</update_frequency>
-        </plugin>
-      </gazebo>
-    </xacro:if>
-    <!-- ROS2 controls -->
-    <ros2_control name="j100_hardware" type="system">
-      <hardware>
-        <xacro:if value="$(arg is_sim)">
-          <plugin>ign_ros2_control/IgnitionSystem</plugin>
-        </xacro:if>
-        <xacro:unless value="$(arg is_sim)">
-          <plugin>clearpath_platform/J100Hardware</plugin>
-        </xacro:unless>
-      </hardware>
-      <joint name="front_left_wheel_joint">
-        <command_interface name="velocity"/>
-        <state_interface name="position"/>
-        <state_interface name="velocity"/>
-      </joint>
-      <joint name="rear_left_wheel_joint">
-        <command_interface name="velocity"/>
-        <state_interface name="position"/>
-        <state_interface name="velocity"/>
-      </joint>
-      <joint name="front_right_wheel_joint">
-        <command_interface name="velocity"/>
-        <state_interface name="position"/>
-        <state_interface name="velocity"/>
-      </joint>
-      <joint name="rear_right_wheel_joint">
-        <command_interface name="velocity"/>
-        <state_interface name="position"/>
-        <state_interface name="velocity"/>
-      </joint>
-    </ros2_control>
   </xacro:macro>
 </robot>

Commit message: Added 35mm standoffs offset for AMD computer
Signed-off-by: Abhishekh Reddy <helloarm@pm.me>

File: honeybee_description/urdf/honeybee_description.urdf.xacro (robot description, xacro)
@@ -25,5 +25,5 @@
   </xacro:fender>
   <xacro:top_plate name="ark_enclosure" model="ark_enclosure" parent_link="default_mount">
-    <origin xyz="0.0 0.0 0.0" rpy="0.0 0.0 0.0"/>
+    <origin xyz="0.0 0.0 0.035" rpy="0.0 0.0 0.0"/> <!-- + 0.035m for Ryzen AI Max standoffs -->
   </xacro:top_plate>
   <!-- Metal enclosure -->
